Commit message: 19/10

File: install/my_robot_description/share/my_robot_description/urdf/common_property.xacro (robot description, xacro)
@@ -1,36 +1 @@
-<?xml version="1.0"?>
-<robot xmlns:xacro="http://ros.org/wiki/xacro">
-    <material name="blue">
-        <color rgba="0 0 0.5 1" />
-    </material>
-    <material name="grey">
-        <color rgba="0.5 0.5 0.5 1" />
-    </material>
-    <xacro:macro name="box_inertia" params="m l w h xyz rpy">
-        <inertial>
-            <origin xyz="${xyz}" rpy="${rpy}" />
-            <mass value="${m}" />
-            <inertia ixx="${(m/12) * (h*h + l*l)}" ixy="0" ixz="0"
-                     iyy="${(m/12) * (w*w + l*l)}" iyz="0"
-                     izz="${(m/12) * (w*w + h*h)}" />
-        </inertial>
-    </xacro:macro>
-    <xacro:macro name="cylinder_inertia" params="m r h xyz rpy">
-        <inertial>
-            <origin xyz="${xyz}" rpy="${rpy}" />
-            <mass value="${m}" />
-            <inertia ixx="${(m/12) * (3*r*r + h*h)}" ixy="0" ixz="0"
-                     iyy="${(m/12) * (3*r*r + h*h)}" iyz="0"
-                     izz="${(m/2) * (r*r)}" />
-        </inertial>
-    </xacro:macro>
-    <xacro:macro name="sphere_inertia" params="m r xyz rpy">
-        <inertial>
-            <origin xyz="${xyz}" rpy="${rpy}" />
-            <mass value="${m}" />
-            <inertia ixx="${(2/5) * m * r * r}" ixy="0" ixz="0"
-                     iyy="${(2/5) * m * r * r}" iyz="0"
-                     izz="${(2/5) * m * r * r}" />
-        </inertial>
-    </xacro:macro>
-</robot>
+/home/dung/ros_ws/src/my_robot_description/urdf/common_property.xacro

File: install/my_robot_description/share/my_robot_description/urdf/lidar_config.xacro (robot description, xacro)
@@ -1,43 +1 @@
-<?xml version="1.0"?>
-<robot xmlns:xacro="http://ros.org/wiki/xacro">
-    <joint name="laser_joint" type="fixed">
-        <parent link="base_link"/>
-        <child link="laser_frame"/>
-        <origin xyz="0 0 0.225" rpy="0 0 0"/>
-    </joint>
-    <link name="laser_frame">
-        <visual>
-            <origin xyz="0 0 0"/>
-            <geometry>
-                <cylinder radius="0.05" length="0.04"/>
-            </geometry>
-        </visual>
-    </link>
-    <gazebo reference="laser_frame">
-        <sensor name="laser" type="ray">
-            <pose> 0 0 0.225 0 0 0 </pose>
-            <visualize>true</visualize>
-            <update_rate>10</update_rate>
-            <ray>
-                <scan>
-                    <horizontal>
-                        <samples>360</samples>
-                        <min_angle>-3.14</min_angle>
-                        <max_angle>3.14</max_angle>
-                    </horizontal>
-                </scan>
-                <range>
-                    <min>0.3</min>
-                    <max>12</max>
-                </range>
-            </ray>
-            <plugin name="laser_controller" filename="libgazebo_ros_ray_sensor.so">
-                <ros>
-                    <argument>~/out:=scan</argument>
-                </ros>
-                <output_type>sensor_msgs/LaserScan</output_type>
-                <frame_name>laser_frame</frame_name>
-            </plugin>
-        </sensor>
-    </gazebo>
-</robot>
+/home/dung/ros_ws/src/my_robot_description/urdf/lidar_config.xacro

File: install/my_robot_description/share/my_robot_description/urdf/mobile_base.xacro (robot description, xacro)
@@ -1,108 +1 @@
-<?xml version="1.0"?>
-<robot xmlns:xacro="http://ros.org/wiki/xacro">
-    <xacro:property name="base_length" value="0.6" />
-    <xacro:property name="base_width" value="0.4" />
-    <xacro:property name="base_height" value="0.2" />
-    <xacro:property name="wheel_radius" value="0.1" />
-    <xacro:property name="wheel_length" value="0.05" />
-    <link name="base_footprint" />
-    <link name="base_link">
-        <visual>
-            <geometry>
-                <box size="${base_length} ${base_width} ${base_height}" />
-            </geometry>
-            <origin xyz="0 0 ${base_height / 2.0}" rpy="0 0 0" />
-            <material name="blue" />
-        </visual>
-        <collision>
-            <geometry>
-                <box size="${base_length} ${base_width} ${base_height}" />
-            </geometry>
-            <origin xyz="0 0 ${base_height / 2.0}" rpy="0 0 0" />
-        </collision>
-        <xacro:box_inertia m="5.0" l="${2*base_length}" w="${2*base_width}" h="${2*base_height}"
-                           xyz="0 0 ${base_height / 2.0}" rpy="0 0 0" />
-    </link>
-    <xacro:macro name="wheel_link" params="prefix">
-        <link name="${prefix}_wheel_link">
-            <visual>
-                <geometry>
-                    <cylinder radius="${wheel_radius}" length="${wheel_length}" />
-                </geometry>
-                <origin xyz="0 0 0" rpy="${pi / 2.0} 0 0" />
-                <material name="grey" />
-            </visual>
-            <collision>
-                <geometry>
-                    <cylinder radius="${wheel_radius}" length="${wheel_length}" />
-                </geometry>
-                <origin xyz="0 0 0" rpy="${pi / 2.0} 0 0" />
-            </collision>
-            <xacro:cylinder_inertia m="1.0" r="${2*wheel_radius}" h="${2*wheel_length}"
-                                    xyz="0 0 0" rpy="${pi / 2.0} 0 0" />
-        </link>
-    </xacro:macro>
-    <xacro:wheel_link prefix="right" />
-    <xacro:wheel_link prefix="left" />
-    <link name="caster_wheel_link">
-        <visual>
-            <geometry>
-                <sphere radius="${wheel_radius / 2.0}" />
-            </geometry>
-            <origin xyz="0 0 0" rpy="0 0 0" />
-            <material name="grey" />
-        </visual>
-        <collision>
-            <geometry>
-                <sphere radius="${wheel_radius / 2.0}" />
-            </geometry>
-            <origin xyz="0 0 0" rpy="0 0 0" />
-        </collision>
-        <xacro:sphere_inertia m="0.5" r="${2*wheel_radius / 2.0}"
-                              xyz="0 0 0" rpy="0 0 0" />
-    </link>
-    <joint name="base_joint" type="fixed">
-        <parent link="base_footprint" />
-        <child link="base_link" />
-        <origin xyz="0 0 ${wheel_radius}" rpy="0 0 0"/>
-    </joint>
-    <joint name="base_right_wheel_joint" type="continuous">
-        <parent link="base_link" />
-        <child link="right_wheel_link" />
-        <origin xyz="${-base_length / 4.0} ${-(base_width + wheel_length) / 2.0} 0" rpy="0 0 0" />
-        <axis xyz="0 1 0" />
-    </joint>
-    <joint name="base_left_wheel_joint" type="continuous">
-        <parent link="base_link" />
-        <child link="left_wheel_link" />
-        <origin xyz="${-base_length / 4.0} ${(base_width + wheel_length) / 2.0} 0" rpy="0 0 0" />
-        <axis xyz="0 1 0" />
-    </joint>
-    <joint name="base_caster_wheel_joint" type="fixed">
-        <parent link="base_link" />
-        <child link="caster_wheel_link" />
-        <origin xyz="${base_length / 3.0} 0 ${-wheel_radius / 2.0}" rpy="0 0 0" />
-    </joint>
-    <link name="imu_link">
-        <inertial>
-            <origin xyz="-0.00552433659106688 0.000168210391520346 0.000514000497342681" rpy="0 0 0" />
-                <mass value="0.000528415362211671" />
-                <inertia
-                ixx="1.46176048428261E-08" ixy="1.40015117949421E-10" ixz="-1.99633872937403E-12"
-                iyy="8.59662482954888E-09" iyz="7.52375112767959E-12"
-                izz="2.30279421279312E-08" />
-        </inertial>
-    <visual>
-        <origin xyz="0 0 0" rpy="0 0 0" />
-    </visual>
-    <collision>
-        <origin xyz="0 0 0" rpy="0 0 0" />
-    </collision>
-    </link>
-    <joint name="imu_joint" type="fixed">
-        <origin xyz="0 0 0.0698986241758014" rpy="0 0 0" />
-        <parent link="base_link" />
-        <child link="imu_link" />
-        <axis xyz="0 0 0" />
-    </joint>
-</robot>
+/home/dung/ros_ws/src/my_robot_description/urdf/mobile_base.xacro

File: install/my_robot_description/share/my_robot_description/urdf/mobile_base_gazebo.xacro (robot description, xacro)
@@ -1,99 +1 @@
-<?xml version="1.0"?>
-<robot name="my_robot" xmlns:xacro="http://ros.org/wiki/xacro">
-    <gazebo reference="base_link">
-        <material>Gazebo/Blue</material>
-    </gazebo>
-    <gazebo reference="caster_wheel_link">
-        <material>Gazebo/Grey</material>
-        <mu1 value="0.1"/>
-        <mu2 value="0.2"/>
-    </gazebo>
-    <gazebo reference="right_wheel_link">
-        <material>Gazebo/Red</material>
-    </gazebo>
-    <gazebo reference="left_wheel_link">
-        <material>Gazebo/Red</material>
-    </gazebo>
-    <!-- <gazebo>
-        <plugin name="gazebo_ros_diff_drive" filename="libgazebo_ros_diff_drive.so">
-            <update_rate>50</update_rate>
-            <left_joint>base_left_wheel_joint</left_joint>
-            <right_joint>base_right_wheel_joint</right_joint>
-            <wheel_separation>0.45</wheel_separation>
-            <wheel_diameter>0.2</wheel_diameter>
-            <command_topic>cmd_vel</command_topic>
-            <publish_odom>true</publish_odom>
-            <publish_odom_tf>true</publish_odom_tf>
-            <publish_wheel_tf>true</publish_wheel_tf>
-            <odometry_topic>odom</odometry_topic>
-            <odometry_frame>odom</odometry_frame>
-            <robot_base_frame>base_footprint</robot_base_frame>
-        </plugin>
-    </gazebo> -->
-    <gazebo>
-        <xacro:if value = "$(arg is_ignition)">
-            <plugin filename= "ign_ros2_control-system" name="ign_ros2_control::IgnitionROS2ControlPlugin">
-                <parameters>$(find myrobot_controller)/config/myrobot_config.yaml</parameters>
-            </plugin>
-            <plugin filename= "ignition-gazebo-imu-system" name="ignition::gazebo::systems::Imu">
-            </plugin>
-        </xacro:if>
-        <xacro:unless value = "$(arg is_ignition)">
-            <plugin filename= "gz_ros2_control-system" name="gz_ros2_control::GazeboSimROS2ControlPlugin">
-                <parameters>$(find myrobot_controller)/config/myrobot_config.yaml</parameters>
-            </plugin>
-            <plugin filename= "gz-sim-imu-system" name="gz::sim::systems::Imu">
-            </plugin>
-        </xacro:unless>
-    </gazebo>
-    <gazebo reference="imu_link">
-        <sensor name = "imu" type = "imu">
-            <always_on>true</always_on>
-            <update_rate>50</update_rate>
-            <gz_frame_id>imu_link</gz_frame_id>
-            <topic>imu</topic>
-            <imu>
-                <angular_velocity>
-                    <x>
-                        <noise type= "gaussian">
-                            <mean>0.0</mean>
-                            <stddev>2e-4</stddev>
-                        </noise>
-                    </x>
-                    <y>
-                        <noise type= "gaussian">
-                            <mean>0.0</mean>
-                            <stddev>2e-4</stddev>
-                        </noise>
-                    </y>
-                    <z>
-                        <noise type= "gaussian">
-                            <mean>0.0</mean>
-                            <stddev>2e-4</stddev>
-                        </noise>
-                    </z>
-                </angular_velocity>
-                <linear_acceleration>
-                    <x>
-                        <noise type= "gaussian">
-                            <mean>0.0</mean>
-                            <stddev>1.7e-2</stddev>
-                        </noise>
-                    </x>
-                    <y>
-                        <noise type= "gaussian">
-                            <mean>0.0</mean>
-                            <stddev>1.7e-2</stddev>
-                        </noise>
-                    </y>
-                    <z>
-                        <noise type= "gaussian">
-                            <mean>0.0</mean>
-                            <stddev>1.7e-2</stddev>
-                        </noise>
-                    </z>
-                </linear_acceleration>
-            </imu>
-        </sensor>
-    </gazebo>
-</robot>
+/home/dung/ros_ws/src/my_robot_description/urdf/mobile_base_gazebo.xacro

File: install/my_robot_description/share/my_robot_description/urdf/my_robot.urdf.xacro (robot description, xacro)
@@ -1,8 +1 @@
-<?xml version="1.0"?>
-<robot name="my_robot" xmlns:xacro="http://ros.org/wiki/xacro">
-    <xacro:arg name="is_ignition" default= "true"/>
-    <xacro:include filename="myrobot_control.xacro"/>
-    <xacro:include filename="common_property.xacro"/>
-    <xacro:include filename="mobile_base.xacro"/>
-    <xacro:include filename="mobile_base_gazebo.xacro"/>
-</robot>
+/home/dung/ros_ws/src/my_robot_description/urdf/my_robot.urdf.xacro

File: install/my_robot_description/share/my_robot_description/urdf/myrobot_control.xacro (robot description, xacro)
@@ -1,31 +1 @@
-<?xml version="1.0"?>
-<robot name="my_robot" xmlns:xacro="http://ros.org/wiki/xacro">
-    <ros2_control name="RobotSystem" type="system">
-        <xacro:if value="$(arg is_ignition)">
-            <hardware>
-                <plugin>ign_ros2_control/IgnitionSystem</plugin>
-            </hardware>
-        </xacro:if>
-        <xacro:unless value="$(arg is_ignition)">
-            <hardware>
-                <plugin>gz_ros2_control/GazeboSimSystem</plugin>
-            </hardware>
-        </xacro:unless>
-        <joint name="base_right_wheel_joint">
-            <command_interface name="velocity">
-                <param name="min">-1</param>
-                <param name="max">1</param>
-            </command_interface>
-            <state_interface name="position"/>
-            <state_interface name="velocity"/>
-        </joint>
-        <joint name="base_left_wheel_joint">
-            <command_interface name="velocity">
-                <param name="min">-1</param>
-                <param name="max">1</param>
-            </command_interface>
-            <state_interface name="position"/>
-            <state_interface name="velocity"/>
-        </joint>
-    </ros2_control>
-</robot>
+/home/dung/ros_ws/src/my_robot_description/urdf/myrobot_control.xacro

File: src/my_robot_description/urdf/lidar_config.xacro (robot description, xacro)
@@ -4,5 +4,5 @@
         <parent link="base_link"/>
         <child link="laser_frame"/>
-        <origin xyz="0 0 0.225" rpy="0 0 0"/>
+        <origin xyz="0 0 0.08" rpy="0 0 0"/>
     </joint>
     <link name="laser_frame">

File: src/my_robot_description/urdf/mobile_base.xacro (robot description, xacro)
@@ -1,9 +1,10 @@
 <?xml version="1.0"?>
-<robot xmlns:xacro="http://ros.org/wiki/xacro">
-    <xacro:property name="base_length" value="0.6" />
+<robot name="my_robot" xmlns:xacro="http://ros.org/wiki/xacro" >
+    <xacro:property name="base_length" value="0.5" />
     <xacro:property name="base_width" value="0.4" />
-    <xacro:property name="base_height" value="0.2" />
-    <xacro:property name="wheel_radius" value="0.1" />
-    <xacro:property name="wheel_length" value="0.05" />
+    <xacro:property name="base_height" value="0.14" />
+    <xacro:property name="wheel_radius" value="0.04" />
+    <xacro:property name="wheel_length" value="0.03" />
+    <xacro:property name="caster_wheel_radius" value="0.005" />
     <link name="base_footprint" />
     <link name="base_link">
@@ -12,5 +13,5 @@
                 <box size="${base_length} ${base_width} ${base_height}" />
             </geometry>
-            <origin xyz="0 0 ${base_height / 2.0}" rpy="0 0 0" />
+            <origin xyz="0 0 0" rpy="0 0 0" />
             <material name="blue" />
         </visual>
@@ -19,8 +20,8 @@
                 <box size="${base_length} ${base_width} ${base_height}" />
             </geometry>
-            <origin xyz="0 0 ${base_height / 2.0}" rpy="0 0 0" />
+            <origin xyz="0 0 0" rpy="0 0 0" />
         </collision>
-        <xacro:box_inertia m="5.0" l="${2*base_length}" w="${2*base_width}" h="${2*base_height}"
-                           xyz="0 0 ${base_height / 2.0}" rpy="0 0 0" />
+        <xacro:box_inertia m="5.0" l="${base_length}" w="${base_width}" h="${base_height}"
+                           xyz="0 0 0" rpy="0 0 0" />
     </link>
     <xacro:macro name="wheel_link" params="prefix">
@@ -39,5 +40,5 @@
                 <origin xyz="0 0 0" rpy="${pi / 2.0} 0 0" />
             </collision>
-            <xacro:cylinder_inertia m="1.0" r="${2*wheel_radius}" h="${2*wheel_length}"
+            <xacro:cylinder_inertia m="0.5" r="${2*wheel_radius}" h="${2*wheel_length}"
                                     xyz="0 0 0" rpy="${pi / 2.0} 0 0" />
         </link>
@@ -48,5 +49,5 @@
         <visual>
             <geometry>
-                <sphere radius="${wheel_radius / 2.0}" />
+                <sphere radius="${2*caster_wheel_radius}" />
             </geometry>
             <origin xyz="0 0 0" rpy="0 0 0" />
@@ -55,9 +56,26 @@
         <collision>
             <geometry>
-                <sphere radius="${wheel_radius / 2.0}" />
+                <sphere radius="${2*caster_wheel_radius}" />
             </geometry>
             <origin xyz="0 0 0" rpy="0 0 0" />
         </collision>
-        <xacro:sphere_inertia m="0.5" r="${2*wheel_radius / 2.0}"
+        <xacro:sphere_inertia m="0.5" r="${2*caster_wheel_radius}"
+                              xyz="0 0 0" rpy="0 0 0" />
+    </link>
+    <link name="caster_wheel_link1">
+        <visual>
+            <geometry>
+                <sphere radius="${2*caster_wheel_radius}" />
+            </geometry>
+            <origin xyz="0 0 0" rpy="0 0 0" />
+            <material name="grey" />
+        </visual>
+        <collision>
+            <geometry>
+                <sphere radius="${2*caster_wheel_radius}" />
+            </geometry>
+            <origin xyz="0 0 0" rpy="0 0 0" />
+        </collision>
+        <xacro:sphere_inertia m="0.5" r="${2*caster_wheel_radius}"
                               xyz="0 0 0" rpy="0 0 0" />
     </link>
@@ -65,10 +83,10 @@
         <parent link="base_footprint" />
         <child link="base_link" />
-        <origin xyz="0 0 ${wheel_radius}" rpy="0 0 0"/>
+        <origin xyz="0 0 ${0.023 + base_height/2.0}" rpy="0 0 0"/>
     </joint>
     <joint name="base_right_wheel_joint" type="continuous">
         <parent link="base_link" />
         <child link="right_wheel_link" />
-        <origin xyz="${-base_length / 4.0} ${-(base_width + wheel_length) / 2.0} 0" rpy="0 0 0" />
+        <origin xyz="0 ${-(base_width - wheel_length) / 2.0} -0.05" rpy="0 0 0" />
         <axis xyz="0 1 0" />
     </joint>
@@ -76,5 +94,5 @@
         <parent link="base_link" />
         <child link="left_wheel_link" />
-        <origin xyz="${-base_length / 4.0} ${(base_width + wheel_length) / 2.0} 0" rpy="0 0 0" />
+        <origin xyz="0 ${(base_width - wheel_length) / 2.0} -0.05" rpy="0 0 0" />
         <axis xyz="0 1 0" />
     </joint>
@@ -82,5 +100,10 @@
         <parent link="base_link" />
         <child link="caster_wheel_link" />
-        <origin xyz="${base_length / 3.0} 0 ${-wheel_radius / 2.0}" rpy="0 0 0" />
+        <origin xyz="0.1611 0 ${-(base_height/ 2.0 + 0.009)}" rpy="0 0 0" />
+    </joint>
+    <joint name="base_caster_wheel_joint1" type="fixed">
+        <parent link="base_link" />
+        <child link="caster_wheel_link1" />
+        <origin xyz="-0.1611 0 ${-(base_height/ 2.0 + 0.009)}" rpy="0 0 0" />
     </joint>
     <link name="imu_link">
@@ -93,16 +116,49 @@
                 izz="2.30279421279312E-08" />
         </inertial>
-    <visual>
-        <origin xyz="0 0 0" rpy="0 0 0" />
-    </visual>
-    <collision>
-        <origin xyz="0 0 0" rpy="0 0 0" />
-    </collision>
+        <visual>
+            <geometry>
+                <box size="0.05 0.05 0.05"/>
+            </geometry>
+            <origin xyz="0 0 0" rpy="0 0 0" />
+        </visual>
+        <collision>
+            <geometry>
+                <box size="0.05 0.05 0.05" />
+            </geometry>
+            <origin xyz="0 0 0" rpy="0 0 0" />
+        </collision>
     </link>
     <joint name="imu_joint" type="fixed">
-        <origin xyz="0 0 0.0698986241758014" rpy="0 0 0" />
+        <origin xyz="0 0 0.08" rpy="0 0 0" />
         <parent link="base_link" />
         <child link="imu_link" />
         <axis xyz="0 0 0" />
     </joint>
+    <link name="laser_link">
+        <inertial>
+            <origin xyz="-0.011945780406062 -0.000381929217680526 -0.0170649378129477" rpy="0 0 0" />
+                <mass value="0.073084435549317" />
+                <inertia
+                ixx="1.96074931730795E-05" ixy="-3.62091076640009E-07" ixz="4.28230084046735E-07"
+                iyy="2.40983835136327E-05" iyz="1.50180909250652E-08"
+                izz="4.14184164228595E-05" />
+        </inertial>
+        <visual>
+            <geometry>
+                <box size="0.05 0.05 0.05"/>
+            </geometry>
+            <origin xyz="0 0 0" rpy="0 0 0" />
+        </visual>
+        <collision>
+            <geometry>
+                <box size="0.1 0.1 0.05" />
+            </geometry>
+            <origin xyz="0 0 0" rpy="0 0 0" />
+        </collision>
+    </link>
+    <joint name="laser_joint" type="fixed">
+        <origin xyz="0 0 0.08" rpy="0 0 0" />
+        <parent link="base_link" />
+        <child link="laser_link" />
+    </joint>
 </robot>
